File: env_sensor.kicad_pcb (KiCad board)
At the start: 2 copper layers, 102.9 x 143 mm, 48 parts, among them J1 E Paper, J10 PWMOUT, J3 Barrel_Jack, J4 LED_OUTPUT, J5 RegSense, J6 I2c, J7 USB_C_Receptacle_USB2.0_16P, J9 DEBUG, Q1 NMOS, Q2 NMOS, Q3 NMOS, U1 MH-Z19B, U3 ESP32-S3-WROOM-1, U4 TXB0104PW, U5 BME280, U6 TPS2065CDBV, U7 AP7361C-33E, Y1 Crystal

Commit message: update
Parts:
- removed C2, C3: 100n, Capacitor_SMD:C_0603_1608Metric
- removed JP2: Default77, Jumper:SolderJumper-3_P1.3mm_Bridged12_RoundedPad1.0x1.5mm
- removed R2: 4.7K, Resistor_SMD:R_0603_1608Metric
- removed R3: 1k, Resistor_SMD:R_0603_1608Metric
- removed U5: BME280, Package_LGA:Bosch_LGA-8_2.5x2.5mm_P0.65mm_ClockwisePinNumbering
- added J11: Register, Connector_PinHeader_2.54mm:PinHeader_1x03_P2.54mm_Vertical, F.Cu at (171.4, 51.6)
- added J12: I2C_Source, Connector_PinHeader_2.54mm:PinHeader_1x04_P2.54mm_Vertical, F.Cu at (166.8, 51.6)
- added J13: I2C_2, Connector_PinSocket_2.54mm:PinSocket_1x04_P2.54mm_Vertical, F.Cu at (155.3, 92.1)
- added J14: I2C_3, Connector_PinSocket_2.54mm:PinSocket_1x04_P2.54mm_Vertical, F.Cu at (159.9, 92.1)
- added J15: MH-Z19, Connector_PinSocket_2.54mm:PinSocket_1x04_P2.54mm_Vertical, F.Cu at (102.6, 51.0)
- added J16: ADCs, Connector_PinSocket_2.54mm:PinSocket_1x04_P2.54mm_Vertical, F.Cu at (141.0, 51.0)
- added J2: RegSense, Connector_PinSocket_2.54mm:PinSocket_1x02_P2.54mm_Vertical, F.Cu at (164.5, 92.1)
- added J6: I2C_1, Connector_PinSocket_2.54mm:PinSocket_1x04_P2.54mm_Vertical, F.Cu at (150.7, 92.1)
- added REF**: MountingHole_3.2mm_M3, MountingHole:MountingHole_3.2mm_M3, F.Cu at (147.2, 110.0)
- added REF**: MountingHole_3.2mm_M3, MountingHole:MountingHole_3.2mm_M3, F.Cu at (182.2, 45.0)
- added REF**: MountingHole_3.2mm_M3, MountingHole:MountingHole_3.2mm_M3, F.Cu at (147.2, 45.0)
- added REF**: MountingHole_3.2mm_M3, MountingHole:MountingHole_3.2mm_M3, F.Cu at (182.2, 110.0)
- J5: value RegSense -> Conn_01x04_Pin; footprint Connector_PinSocket_2.54mm:PinSocket_1x02_P2.54mm_Vertical -> Connector_PinHeader_2.54mm:PinHeader_1x04_P2.54mm_Vertical
- Q1, Q2, Q3: footprint env-sensor:SOT-23 -> env-sensor:TO-252
- R1: value 4.7K -> 1k
- moved U1 45.7 mm to (179.6, 71.4)
- moved R1 33.3 mm to (164.2, 98.2)
- moved J6 30.1 mm to (134.6, 81.0), turned to -90 degrees
- moved C1 17.9 mm to (127.1, 86.0), turned to 180 degrees
- moved J3 17.2 mm to (130.1, 99.6)
- moved J4 16.2 mm to (119.9, 108.1), turned to -90 degrees
- moved Q1 16.0 mm to (125.6, 93.2), turned to -90 degrees
- moved J1 15.8 mm to (104.6, 85.6), turned to 0 degrees
- moved Q3 12.1 mm to (111.2, 101.4), turned to -90 degrees
- moved Q2 9.61 mm to (118.4, 97.3), turned to -90 degrees
- moved C4 7.86 mm to (119.9, 90.1), turned to 0 degrees
- moved J5 7.24 mm to (145.0, 51.0), turned to 0 degrees
- moved C12 6.98 mm to (118.5, 79.8), turned to 90 degrees
- moved D1 6.18 mm to (106.5, 77.0)
- moved D2 6.14 mm to (106.5, 80.6)
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Connections:
- J5 pad 1: GND -> /sensor/v5v
- J5 pad 2: temp -> /sensor/UART(d2u)
- R1 pad 1: v3v -> /sensor/v3v
- R1 pad 2: SCL -> /sensor/reg
- U1 pad 2: RX(ESP_DOWN) -> /sensor/UART(u2d)
- U1 pad 3: TX(ESP_UP) -> /sensor/UART(d2u)
- U1 pad 6: v5v -> /sensor/v5v
- U1 pad 7: GND -> /sensor/GND
- U3 pad 10: LED_C2 -> LED_C1
- U3 pad 11: LED_C3 -> LED_C2
- U3 pad 12: LED_C1 -> LED_C3
- U3 pad 15: SCL -> SPI_MOSI
- U3 pad 16: SDA -> SPI_SCLK
- U3 pad 17: SPI_MOSI -> EPD_ChipSelect
- U3 pad 18: SPI_SCLK -> EPD_DataControl
- U3 pad 19: EPD_ChipSelect -> EPD_RST
- U3 pad 20: EPD_DataControl -> EPD_BackLight
- U3 pad 21: EPD_RST -> SDA
- U3 pad 22: EPD_BackLight -> SCL
- U3 pad 23: AD0 -> AD3
- U3 pad 24: AD1 -> AD2
- U3 pad 25: AD2 -> AD1
- U3 pad 26: AD3 -> AD0
- U3 pad 38: unconnected-(U3-IO2-Pad38) -> adc2
- U3 pad 39: temp -> adc1
Routing:
- net v3v: track 6.61 -> 130.0 mm, vias 1 -> 6
- net EPD_BackLight: track 0.00 -> 45.7 mm
- net EPD_RST: track 0.00 -> 43.4 mm
- net EPD_DataControl: track 0.00 -> 41.0 mm
- net EPD_ChipSelect: track 0.00 -> 40.0 mm
- net SPI_SCLK: track 0.00 -> 38.1 mm
- net SPI_MOSI: track 0.00 -> 37.2 mm
- net LED_C1: track 0.00 -> 35.6 mm, vias 0 -> 2
- net LED_C2: track 0.00 -> 33.3 mm, vias 0 -> 2
- net LED_C3: track 0.00 -> 32.7 mm, vias 0 -> 2
- net LED_V1: track 0.00 -> 17.1 mm
- net SCL: track 0.00 -> 17.0 mm
- net SDA: track 0.00 -> 16.4 mm
- net v12: track 0.00 -> 14.6 mm
- net AD3: track 0.00 -> 13.8 mm
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- added copper zone on F.Cu, net VCC
Other:
- board size 102.9 x 143 mm -> 146 x 143 mm

Commit message: fin
Parts:
- added J17: Conn_01x04_Pin, Connector_PinHeader_2.54mm:PinHeader_1x04_P2.54mm_Vertical, F.Cu at (186.0, 51.0)
- added R2: 1k, Resistor_THT:R_Axial_DIN0207_L6.3mm_D2.5mm_P10.16mm_Horizontal, F.Cu at (181.3, 69.7)
- J11: value Register -> Reg2; footprint Connector_PinHeader_2.54mm:PinHeader_1x03_P2.54mm_Vertical -> Connector_PinSocket_2.54mm:PinSocket_1x02_P2.54mm_Vertical
- J2: value RegSense -> Reg1
- R1: footprint Resistor_SMD:R_0603_1608Metric -> Resistor_THT:R_Axial_DIN0207_L6.3mm_D2.5mm_P10.16mm_Horizontal
- moved R1 47.3 mm to (185.1, 55.7), turned to -90 degrees
- moved U1 32.3 mm to (151.8, 55.0), turned to 90 degrees
- moved J12 32.0 mm to (179.6, 81.0), turned to -90 degrees
- moved J2 28.6 mm to (185.1, 72.3), turned to 180 degrees
- moved J11 26.4 mm to (181.3, 76.1), turned to 180 degrees
- moved J5 2.55 mm to (147.6, 51.0)
- moved REF** 1.84 mm to (149.0, 110.0)
- moved REF** 1.84 mm to (184.0, 45.0)
- moved REF** 1.84 mm to (149.0, 45.0)
- moved REF** 1.84 mm to (184.0, 110.0)
Connections:
- J11 pad 1: /sensor/v3v -> /sensor/GND
- J11 pad 2: /sensor/reg -> /sensor/adc2
- J16 pad 2: GND -> adc1
- J16 pad 3: adc1 -> adc2
- J16 pad 4: adc2 -> GND
- J2 pad 2: /sensor/reg -> /sensor/adc1
- R1 pad 1: /sensor/v3v -> /sensor/adc_v3v
- R1 pad 2: /sensor/reg -> /sensor/adc1
Routing:
- net /sensor/v5v: track 0.00 -> 42.3 mm
- net /sensor/v3v: track 0.00 -> 36.9 mm
- net /sensor/SCL: track 0.00 -> 29.4 mm
- net /sensor/SDA: track 0.00 -> 25.8 mm
- net /sensor/adc2: track 0.00 -> 24.9 mm
- net /sensor/adc1: track 0.00 -> 22.6 mm
- net /sensor/UART(u2d): track 0.00 -> 16.8 mm
- net /sensor/UART(d2u): track 0.00 -> 13.8 mm
- net /sensor/adc_v3v: track 0.00 -> 10.9 mm
- net GND: vias 14 -> 16
- net /sensor/GND: vias 0 -> 11
- added copper zone on B.Cu, net /sensor/GND
- added copper zone on F.Cu, net /sensor/GND
Other:
- board size 146 x 143 mm -> 147.9 x 143 mm
