File: env_sensor.kicad_sch (KiCad schematic)
At the start: 47 parts, among them J1 E Paper, J10 PWMOUT, J3 Barrel_Jack, J4 LED_OUTPUT, J5 RegSense, J6 I2c, J7 USB_C_Receptacle_USB2.0_16P, J8 v5_v3, J9 DEBUG, Q1 NMOS, Q2 NMOS, Q3 NMOS, SW1 EN, SW2 BOOT, U1 MH-Z19B, U3 ESP32-S3-WROOM-1, U4 TXB0104PW, U5 BME280, U6 TPS2065CDBV, U7 AP7361C-33E, Y1 Crystal

Commit message: update
Parts:
- removed C2, C3: 100n, Capacitor_SMD:C_0603_1608Metric, symbol Device:C
- removed J5: RegSense, Connector_PinSocket_2.54mm:PinSocket_1x02_P2.54mm_Vertical, symbol Connector:Conn_01x02_Pin
- removed J6: I2c, Connector_PinSocket_2.54mm:PinSocket_1x04_P2.54mm_Vertical, symbol Connector:Conn_01x04_Socket
- removed JP2: Default77, Jumper:SolderJumper-3_P1.3mm_Bridged12_RoundedPad1.0x1.5mm, symbol Jumper:SolderJumper_3_Bridged12
- removed R1, R2: 4.7K, Resistor_SMD:R_0603_1608Metric, symbol Device:R
- removed R3: 1k, Resistor_SMD:R_0603_1608Metric, symbol Device:R
- removed U1: MH-Z19B, mh-z19b:Winsen_MH-Z19B, symbol mh_z19b:MH-Z19B
- removed U5: BME280, Package_LGA:Bosch_LGA-8_2.5x2.5mm_P0.65mm_ClockwisePinNumbering, symbol Sensor:BME280
- added J15: MH-Z19, Connector_PinSocket_2.54mm:PinSocket_1x04_P2.54mm_Vertical, symbol Connector:Conn_01x04_Socket
- added J16: ADCs, Connector_PinSocket_2.54mm:PinSocket_1x04_P2.54mm_Vertical, symbol Connector:Conn_01x04_Socket
- Q1, Q2: footprint env-sensor:SOT-23 -> env-sensor:TO-252
- Q3: footprint env-sensor:SOT-23 -> env-sensor:TO-252; LCSC C916396 -> C557932
Connections:
- net AD0: now also U3.26 (IO45); no longer U3.23 (IO21)
- net AD1: now also U3.25 (IO48); no longer U3.24 (IO47)
- net AD2: now also U3.24 (IO47); no longer U3.25 (IO48)
- net AD3: now also U3.23 (IO21); no longer U3.26 (IO45)
- net EPD_BackLight: now also U3.20 (IO12); no longer U3.22 (IO14)
- net EPD_ChipSelect: now also U3.17 (IO9); no longer U3.19 (IO11)
- net EPD_DataControl: now also U3.18 (IO10); no longer U3.20 (IO12)
- net EPD_RST: now also U3.19 (IO11); no longer U3.21 (IO13)
- net GND: now also J15.2 (Pin_2), J16.2 (Pin_2)
- net LED_C1: now also U3.10 (IO17); no longer U3.12 (IO8)
- net LED_C2: now also U3.11 (IO18); no longer U3.10 (IO17)
- net LED_C3: now also U3.12 (IO8); no longer U3.11 (IO18)
- net RX(ESP_DOWN): now also J15.3 (Pin_3)
- net SCL: now also U3.22 (IO14); no longer U3.15 (IO3)
- net SDA: now also U3.21 (IO13); no longer U3.16 (IO46)
- net SPI_MOSI: now also U3.15 (IO3); no longer U3.17 (IO9)
- net SPI_SCLK: now also U3.16 (IO46); no longer U3.18 (IO10)
- net TX(ESP_UP): now also J15.4 (Pin_4)
- net v3v: now also J15.1 (Pin_1), J16.1 (Pin_1)
- net adc2: now reaches U3.38 (IO2)
- net adc2: now also J16.4 (Pin_4)
- net temp renamed adc1
- net adc1: now also J16.3 (Pin_3)
- no-connect marks 6 -> 3
Other:
- added sheet sensor (sensor.kicad_sch)
- note removed: "I2C"
- note removed: "サーミスタ回路"
- moved on the sheet: J9

Commit message: fin
Connections:
- net GND: now also J16.4 (Pin_4); no longer J16.2 (Pin_2)
- net adc1: now also J16.2 (Pin_2); no longer J16.3 (Pin_3)
- net adc2: now also J16.3 (Pin_3); no longer J16.4 (Pin_4)
Changed lines of the file:
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@@
+		)
+	)
+	(global_label "adc2"
+		(shape input)
+		(at 31.75 173.99 180)
+		(fields_autoplaced yes)
+		(effects
+			(font
+				(size 1.27 1.27)
+			)
+			(justify right)
+		)
+		(property "Intersheetrefs" "${INTERSHEET_REFS}"
+			(at 24.1687 173.99 0)
+			(effects
+				(font
+					(size 1.27 1.27)
+				)
+				(justify right)
+				(hide yes)
+			)
 		)
 	)
@@
 		)
 	)
-	(global_label "adc1"
-		(shape input)
-		(at 31.75 173.99 180)
-		(fields_autoplaced yes)
-		(effects
-			(font
-				(size 1.27 1.27)
-			)
-			(justify right)
-		)
-		(property "Intersheetrefs" "${INTERSHEET_REFS}"
-			(at 24.1687 173.99 0)
-			(effects
-				(font
-					(size 1.27 1.27)
-				)
-				(justify right)
-				(hide yes)
-			)
-		)
-	)
 	(global_label "GND"
 		(shape input)
@@
 		)
 	)
-	(global_label "adc2"
-		(shape input)
-		(at 31.75 176.53 180)
-		(fields_autoplaced yes)
-		(effects
-			(font
-				(size 1.27 1.27)
-			)
-			(justify right)
-		)
-		(property "Intersheetrefs" "${INTERSHEET_REFS}"
-			(at 24.1687 176.53 0)
-			(effects
-				(font
-					(size 1.27 1.27)
-				)
-				(justify right)
-				(hide yes)
-			)
-		)
-	)
 	(global_label "LED_C1"
 		(shape input)
@@
 		)
 	)
+	(global_label "v5v"
+		(shape input)
+		(at 134.62 16.51 180)
+		(fields_autoplaced yes)
+		(effects
+			(font
+				(size 1.27 1.27)
+			)
+			(justify right)
+		)
+		(property "Intersheetrefs" "${INTERSHEET_REFS}"
+			(at 128.4901 16.51 0)
+			(effects
+				(font
+					(size 1.27 1.27)
+				)
+				(justify right)
+				(hide yes)
+			)
+		)
+	)
+	(global_label "adc1"
+		(shape input)
+		(at 31.75 171.45 180)
+		(fields_autoplaced yes)
+		(effects
+			(font
+				(size 1.27 1.27)
+			)
+			(justify right)
+		)
+		(property "Intersheetrefs" "${INTERSHEET_REFS}"
+			(at 24.1687 171.45 0)
+			(effects
+				(font
+					(size 1.27 1.27)
+				)
+				(justify right)
+				(hide yes)
+			)
+		)
+	)
+	(global_label "EPD_ChipSelect"
+		(shape input)
+		(at 191.77 151.13 180)
+		(fields_autoplaced yes)
+		(effects
+			(font
+				(size 1.27 1.27)
+			)
+			(justify right)
+		)
+		(property "Intersheetrefs" "${INTERSHEET_REFS}"
+			(at 174.0892 151.13 0)
+			(effects
+				(font
+					(size 1.27 1.27)
+				)
+				(justify right)
+				(hide yes)
+			)
+		)
+	)
 	(global_label "GND"
 		(shape input)
-		(at 31.75 171.45 180)
-		(fields_autoplaced yes)
-		(effects
-			(font
-				(size 1.27 1.27)
-			)
-			(justify right)
-		)
-		(property "Intersheetrefs" "${INTERSHEET_REFS}"
-			(at 24.8943 171.45 0)
-			(effects
-				(font
-					(size 1.27 1.27)
-				)
-				(justify right)
-				(hide yes)
-			)
-		)
-	)
-	(global_label "v5v"
-		(shape input)
-		(at 134.62 16.51 180)
-		(fields_autoplaced yes)
-		(effects
-			(font
-				(size 1.27 1.27)
-			)
-			(justify right)
-		)
-		(property "Intersheetrefs" "${INTERSHEET_REFS}"
-			(at 128.4901 16.51 0)
-			(effects
-				(font
-					(size 1.27 1.27)
-				)
-				(justify right)
-				(hide yes)
-			)
-		)
-	)
-	(global_label "EPD_ChipSelect"
-		(shape input)
-		(at 191.77 151.13 180)
-		(fields_autoplaced yes)
-		(effects
-			(font
-				(size 1.27 1.27)
-			)
-			(justify right)
-		)
-		(property "Intersheetrefs" "${INTERSHEET_REFS}"
-			(at 174.0892 151.13 0)
-			(effects
-				(font
+		(at 31.75 176.53 180)
+		(fields_autoplaced yes)
+		(effects
+			(font
+				(size 1.27 1.27)
+			)
+			(justify right)
+		)
+		(property "Intersheetrefs" "${INTERSHEET_REFS}"
+			(at 24.8943 176.53 0)
+			(effects
+				(font

Commit message: update lib for switch and fix DRCs
Parts:
- SW1, SW2: footprint (none) -> paripalpp_button:TVAF06-A020B-R
Changed lines of the file:
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@@
 			)
 		)
-		(property "Footprint" ""
+		(property "Footprint" "paripalpp_button:TVAF06-A020B-R"
 			(at 140.97 115.57 0)
 			(effects
@@
 			)
 		)
-		(property "Footprint" ""
+		(property "Footprint" "paripalpp_button:TVAF06-A020B-R"
 			(at 132.08 114.3 0)
 			(effects

Commit message: update
Parts:
- added J18: Conn_01x02_Pin, Connector_PinHeader_2.54mm:PinHeader_1x02_P2.54mm_Vertical, symbol Connector:Conn_01x02_Pin
- J9: footprint Connector_PinSocket_2.54mm:PinSocket_1x05_P2.54mm_Vertical -> Connector_PinHeader_2.54mm:PinHeader_1x05_P2.54mm_Vertical
Connections:
- net GND: now also J18.2 (Pin_2)
- net RX(ESP_DOWN): now also J15.4 (Pin_4); no longer J15.3 (Pin_3)
- net TX(ESP_UP): now also J15.3 (Pin_3); no longer J15.4 (Pin_4)
- net VCC: now also J15.1 (Pin_1), J8.1 (Pin_1)
- net v3v: no longer J15.1 (Pin_1)
- net v5v: now also J18.1 (Pin_1); no longer J8.1 (Pin_1)
- net VServo: now reaches C6.1, J10.2 (Pin_2), J8.2 (Pin_2), U4.14 (VCCB)
Other:
- moved on the sheet: C10, C11, C12, C13, C14, C6, C7, C8, C9, D1, D2, D3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

Commit message: update BOM
Parts:
- C7, C9: LCSC (none) -> C1853272
- D1, D2, D3: LCSC C86598 -> C123070
- R4: LCSC (none) -> C25804
- R5, R6: LCSC (none) -> C23186
- U6: LCSC (none) -> C353882
- U7: LCSC (none) -> C500795
Changed lines of the file:
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@@
 			)
 		)
-		(property "LCSC" ""
+		(property "LCSC" "C1853272"
 			(at 53.34 148.59 90)
 			(effects
@@
 			)
 		)
-		(property "LCSC" ""
+		(property "LCSC" "C25804"
 			(at 144.78 41.91 0)
 			(effects
@@
 			)
 		)
+		(property "LCSC" "C500795"
+			(at 109.22 152.4 0)
+			(effects
+				(font
+					(size 1.27 1.27)
+				)
+				(hide yes)
+			)
+		)
 		(pin "1"
 		)
@@
 			)
 		)
-		(property "LCSC" ""
+		(property "LCSC" "C23186"
 			(at 60.96 172.72 0)
 			(effects
@@
 			)
 		)
-		(property "LCSC" "C86598"
+		(property "LCSC" "C123070"
 			(at 109.22 143.51 0)
 			(effects
@@
 			)
 		)
-		(property "LCSC" ""
+		(property "LCSC" "C1853272"
 			(at 175.26 41.91 90)
 			(effects
@@
 			)
 		)
+		(property "LCSC" "C353882"
+			(at 71.12 154.94 0)
+			(effects
+				(font
+					(size 1.27 1.27)
+				)
+				(hide yes)
+			)
+		)
 		(pin "1"
 		)
@@
 			)
 		)
-		(property "LCSC" "C86598"
+		(property "LCSC" "C123070"
 			(at 87.63 152.4 0)
 			(effects
@@
 			)
 		)
-		(property "LCSC" ""
+		(property "LCSC" "C23186"
 			(at 69.85 172.72 0)
 			(effects
@@
 					(size 1.27 1.27)
 				)
-				(hide yes)
 			)
 		)
-		(property "LCSC" "C86598"
+		(property "LCSC" "C123070"
 			(at 87.63 144.78 0)
 			(effects

Commit message: ok
Parts:
- added J6: ADCs, Connector_PinSocket_2.54mm:PinSocket_1x04_P2.54mm_Vertical, symbol Connector:Conn_01x04_Socket
- C1, C4, C5: LCSC C14663 -> C1525
- C10, C6: LCSC C5137578 -> C19702
- C11: LCSC C5137578 -> C363553
- C12: LCSC C5137578 -> C380326
- C13, C14: LCSC (none) -> C5360831
- C7, C9: LCSC C1853272 -> C1525
- C8: LCSC (none) -> C307477
- J7: footprint Connector_USB:USB_C_Receptacle_GCT_USB4105-xx-A_16P_TopMnt_Horizontal -> Connector_USB:USB_C_Receptacle_GCT_USB4085; LCSC (none) -> C7095263
- Y1: LCSC (none) -> C1669858
Connections:
- net GND: now also J6.2 (Pin_2)
- net RX(ESP_DOWN): now also J15.3 (Pin_3), U3.5 (IO5); no longer J15.4 (Pin_4), U3.4 (IO4)
- net SCL: now also J6.3 (Pin_3)
- net SDA: now also J6.4 (Pin_4)
- net TX(ESP_UP): now also J15.4 (Pin_4), U3.4 (IO4); no longer J15.3 (Pin_3), U3.5 (IO5)
- net v3v: now also J6.1 (Pin_1)

Commit message: update
Parts:
- C8: LCSC C307477 -> C136131
- J10, J18, J9, U3: now left out of the parts list
- Q1, Q2: LCSC C916396 -> C557932
Connections:
- net U6_OUT: now reaches C9.2, J7.A4 (VBUS), J7.A9 (VBUS), J7.B4 (VBUS), J7.B9 (VBUS), U6.4 (EN), U6.5 (IN)
Other:
- moved on the sheet: C9
Changed lines of the file:
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@@
 	)
 	(junction
+		(at 50.8 152.4)
+		(diameter 0)
+		(color 0 0 0 0)
+	)
+	(junction
 		(at 171.45 41.91)
 		(diameter 0)
@@
 	(wire
 		(pts
-			(xy 82.55 162.56) (xy 82.55 152.4)
-		)
-		(stroke
-			(width 0)
-			(type default)
-		)
-	)
-	(wire
-		(pts
 			(xy 53.34 66.04) (xy 57.15 66.04)
 		)
@@
 	(wire
 		(pts
-			(xy 53.34 143.51) (xy 53.34 144.78)
-		)
-		(stroke
-			(width 0)
-			(type default)
-		)
-	)
-	(wire
-		(pts
 			(xy 40.64 114.3) (xy 43.18 114.3)
 		)
@@
 	(wire
 		(pts
-			(xy 53.34 152.4) (xy 49.53 152.4)
+			(xy 53.34 152.4) (xy 50.8 152.4)
 		)
 		(stroke
@@
 	(wire
 		(pts
+			(xy 82.55 152.4) (xy 82.55 162.56)
+		)
+		(stroke
+			(width 0)
+			(type default)
+		)
+	)
+	(wire
+		(pts
 			(xy 50.8 167.64) (xy 49.53 167.64)
 		)
@@
 	(wire
 		(pts
+			(xy 57.15 142.24) (xy 53.34 142.24)
+		)
+		(stroke
+			(width 0)
+			(type default)
+		)
+	)
+	(wire
+		(pts
 			(xy 186.69 92.71) (xy 187.96 92.71)
 		)
@@
 	(wire
 		(pts
+			(xy 53.34 142.24) (xy 53.34 143.51)
+		)
+		(stroke
+			(width 0)
+			(type default)
+		)
+	)
+	(wire
+		(pts
 			(xy 236.22 116.84) (xy 245.11 116.84)
 		)
@@
 	(wire
 		(pts
+			(xy 53.34 151.13) (xy 53.34 152.4)
+		)
+		(stroke
+			(width 0)
+			(type default)
+		)
+	)
+	(wire
+		(pts
 			(xy 236.22 134.62) (xy 236.22 133.35)
 		)
@@
 	(wire
 		(pts
+			(xy 50.8 154.94) (xy 50.8 152.4)
+		)
+		(stroke
+			(width 0)
+			(type default)
+		)
+	)
+	(wire
+		(pts
 			(xy 234.95 27.94) (xy 237.49 27.94)
 		)
@@
 		)
 	)
+	(wire
+		(pts
+			(xy 50.8 152.4) (xy 49.53 152.4)
+		)
+		(stroke
+			(width 0)
+			(type default)
+		)
+	)
 	(polyline
 		(pts
@@
 	(wire
 		(pts
+			(xy 52.07 154.94) (xy 50.8 154.94)
+		)
+		(stroke
+			(width 0)
+			(type default)
+		)
+	)
+	(wire
+		(pts
 			(xy 187.96 69.85) (xy 186.69 69.85)
 		)
@@
 		)
 	)
+	(label "U6_OUT"
+		(at 52.07 154.94 0)
+		(fields_autoplaced yes)
+		(effects
+			(font
+				(size 1.27 1.27)
+			)
+			(justify left bottom)
+		)
+	)
 	(label "VServo"
 		(at 250.19 114.3 0)
@@
 		(unit 1)
 		(exclude_from_sim no)
-		(in_bom yes)
+		(in_bom no)
 		(on_board yes)
 		(dnp no)
@@
 	(symbol
 		(lib_id "Device:C")
-		(at 53.34 148.59 0)
+		(at 53.34 147.32 0)
 		(unit 1)
 		(exclude_from_sim no)
@@
 		(dnp no)
 		(property "Reference" "C9"
-			(at 60.198 147.574 0)
+			(at 60.198 146.304 0)
 			(effects
 				(font
@@
 		)
 		(property "Value" "0.1u/10v"
-			(at 60.198 149.86 0)
+			(at 60.198 148.59 0)
 			(effects
 				(font
@@
 		)
 		(property "Footprint" "Capacitor_SMD:C_0603_1608Metric"
-			(at 54.3052 152.4 0)
+			(at 54.3052 151.13 0)
 			(effects
 				(font
@@
 		)
 		(property "Datasheet" "~"
-			(at 53.34 148.59 0)
+			(at 53.34 147.32 0)
 			(effects
 				(font
@@
 		)
 		(property "Description" ""
-			(at 53.34 148.59 0)
+			(at 53.34 147.32 0)
 			(effects
 				(font
@@
 		)
 		(property "LCSC" "C1525"
-			(at 53.34 148.59 90)
+			(at 53.34 147.32 90)
 			(effects
 				(font
@@
 		(unit 1)
 		(exclude_from_sim no)
-		(in_bom yes)
+		(in_bom no)
 		(on_board yes)
 		(dnp no)
@@
 		(exclude_from_sim no)
 		(in_bom no)
-		(on_board no)
+		(on_board yes)
 		(dnp no)
 		(fields_autoplaced yes)
@@
 	(symbol
 		(lib_id "power:GND")
-		(at 53.34 143.51 180)
+		(at 57.15 142.24 90)
 		(unit 1)
 		(exclude_from_sim no)
@@
 		(fields_autoplaced yes)
 		(property "Reference" "#PWR010"
-			(at 53.34 137.16 0)
+			(at 63.5 142.24 0)
 			(effects
 				(font
@@
 		)
 		(property "Value" "GND"
-			(at 53.34 138.43 0)
+			(at 60.96 142.2399 90)
 			(effects
 				(font
 					(size 1.27 1.27)
 				)
+				(justify right)
 			)
 		)
 		(property "Footprint" ""
-			(at 53.34 143.51 0)
+			(at 57.15 142.24 0)
 			(effects
 				(font
@@
 		)
 		(property "Datasheet" ""
-			(at 53.34 143.51 0)
+			(at 57.15 142.24 0)
 			(effects
 				(font
@@
 		)
 		(property "Description" "Power symbol creates a global label with name \"GND\" , ground"
-			(at 53.34 143.51 0)
+			(at 57.15 142.24 0)
 			(effects
 				(font
@@
 			)
 		)
-		(property "LCSC" "C916396"
+		(property "LCSC" "C557932"
 			(at 50.8 71.12 0)
 			(effects
@@
 			)
 		)
-		(property "LCSC" "C916396"
+		(property "LCSC" "C557932"
 			(at 50.8 45.72 0)
 			(effects
@@
 		(exclude_from_sim no)
 		(in_bom no)
-		(on_board no)
+		(on_board yes)
 		(dnp no)
 		(fields_autoplaced yes)
@@
 		(unit 1)
 		(exclude_from_sim no)
-		(in_bom yes)
+		(in_bom no)
 		(on_board yes)
 		(dnp no)
@@
 			)
 		)
-		(property "LCSC" "C307477"
+		(property "LCSC" "C136131"
 			(at 144.78 53.34 90)
 			(effects
@@
 		(unit 1)
 		(exclude_from_sim no)
-		(in_bom yes)
+		(in_bom no)
 		(on_board yes)
 		(dnp no)
@@
 		(on_board yes)
 		(dnp no)
-		(fields_autoplaced yes)
 		(property "Reference" "D2"
 			(at 87.9475 138.43 0)
@@
 		)
 		(property "Value" "D_Schottky"
-			(at 87.9475 140.97 0)
+			(at 88.138 140.716 0)
 			(effects
 				(font
@@
 		)
 		(property "Description" "Schottky diode"
-			(at 87.63 144.78 0)
+			(at 89.916 142.494 0)
 			(effects
 				(font

Commit message: update
Connections:
- net IO19 renamed USB_D-
- net IO20 renamed USB_D+
Other:
- moved on the sheet: J7
Changed lines of the file:
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@@
 	)
 	(junction
-		(at 50.8 152.4)
-		(diameter 0)
-		(color 0 0 0 0)
-	)
-	(junction
 		(at 171.45 41.91)
 		(diameter 0)
@@
 	(wire
 		(pts
-			(xy 50.8 165.1) (xy 49.53 165.1)
+			(xy 40.64 165.1) (xy 39.37 165.1)
 		)
 		(stroke
@@
 	(wire
 		(pts
-			(xy 53.34 152.4) (xy 50.8 152.4)
-		)
-		(stroke
-			(width 0)
-			(type default)
-		)
-	)
-	(wire
-		(pts
 			(xy 259.08 134.62) (xy 262.89 134.62)
 		)
@@
 	(wire
 		(pts
-			(xy 49.53 160.02) (xy 60.96 160.02)
+			(xy 39.37 160.02) (xy 60.96 160.02)
 		)
 		(stroke
@@
 	(wire
 		(pts
-			(xy 50.8 167.64) (xy 49.53 167.64)
+			(xy 40.64 167.64) (xy 39.37 167.64)
 		)
 		(stroke
@@
 	(wire
 		(pts
+			(xy 39.37 170.18) (xy 40.64 170.18)
+		)
+		(stroke
+			(width 0)
+			(type default)
+		)
+	)
+	(wire
+		(pts
 			(xy 236.22 123.19) (xy 236.22 116.84)
 		)
@@
 	(wire
 		(pts
-			(xy 50.8 172.72) (xy 49.53 172.72)
+			(xy 40.64 172.72) (xy 39.37 172.72)
 		)
 		(stroke
@@
 	(wire
 		(pts
-			(xy 50.8 154.94) (xy 50.8 152.4)
-		)
-		(stroke
-			(width 0)
-			(type default)
-		)
-	)
-	(wire
-		(pts
 			(xy 234.95 27.94) (xy 237.49 27.94)
 		)
@@
 	(wire
 		(pts
-			(xy 50.8 152.4) (xy 49.53 152.4)
+			(xy 39.37 152.4) (xy 53.34 152.4)
 		)
 		(stroke
@@
 	(wire
 		(pts
-			(xy 49.53 157.48) (xy 59.69 157.48)
+			(xy 39.37 157.48) (xy 59.69 157.48)
 		)
 		(stroke
@@
 	(wire
 		(pts
-			(xy 50.8 170.18) (xy 49.53 170.18)
-		)
-		(stroke
-			(width 0)
-			(type default)
-		)
-	)
-	(wire
-		(pts
 			(xy 53.34 76.2) (xy 53.34 78.74)
 		)
@@
 	(wire
 		(pts
-			(xy 52.07 154.94) (xy 50.8 154.94)
-		)
-		(stroke
-			(width 0)
-			(type default)
-		)
-	)
-	(wire
-		(pts
 			(xy 187.96 69.85) (xy 186.69 69.85)
 		)
@@
 	)
 	(label "U6_OUT"
-		(at 52.07 154.94 0)
+		(at 45.72 152.4 0)
 		(fields_autoplaced yes)
 		(effects
@@
 		)
 	)
-	(global_label "IO20"
+	(global_label "USB_D+"
 		(shape bidirectional)
 		(at 187.96 67.31 0)
@@
 		)
 	)
-	(global_label "IO19"
+	(global_label "USB_D-"
 		(shape bidirectional)
-		(at 50.8 167.64 0)
+		(at 40.64 167.64 0)
 		(fields_autoplaced yes)
 		(effects
@@
 		)
 		(property "Intersheetrefs" "${INTERSHEET_REFS}"
-			(at 59.2508 167.64 0)
+			(at 49.0908 167.64 0)
 			(effects
 				(font
@@
 		)
 	)
-	(global_label "IO19"
+	(global_label "USB_D-"
 		(shape bidirectional)
 		(at 187.96 64.77 0)
@@
 		)
 	)
-	(global_label "IO20"
+	(global_label "USB_D+"
 		(shape bidirectional)
-		(at 50.8 172.72 0)
+		(at 40.64 172.72 0)
 		(fields_autoplaced yes)
 		(effects
@@
 		)
 		(property "Intersheetrefs" "${INTERSHEET_REFS}"
-			(at 59.2508 172.72 0)
+			(at 49.0908 172.72 0)
 			(effects
 				(font
@@
 		)
 	)
-	(global_label "IO19"
+	(global_label "USB_D-"
 		(shape bidirectional)
-		(at 50.8 165.1 0)
+		(at 40.64 165.1 0)
 		(fields_autoplaced yes)
 		(effects
@@
 		)
 		(property "Intersheetrefs" "${INTERSHEET_REFS}"
-			(at 59.2508 165.1 0)
+			(at 49.0908 165.1 0)
 			(effects
 				(font
@@
 		)
 	)
-	(global_label "IO20"
+	(global_label "USB_D+"
 		(shape bidirectional)
-		(at 50.8 170.18 0)
+		(at 40.64 170.18 0)
 		(fields_autoplaced yes)
 		(effects
@@
 		)
 		(property "Intersheetrefs" "${INTERSHEET_REFS}"
-			(at 59.2508 170.18 0)
+			(at 49.0908 170.18 0)
 			(effects
 				(font
@@
 	(symbol
 		(lib_id "power:GND")
-		(at 26.67 190.5 0)
+		(at 16.51 190.5 0)
 		(unit 1)
 		(exclude_from_sim no)
@@
 		(fields_autoplaced yes)
 		(property "Reference" "#PWR02"
-			(at 26.67 196.85 0)
+			(at 16.51 196.85 0)
 			(effects
 				(font
@@
 		)
 		(property "Value" "GND"
-			(at 26.67 195.58 0)
+			(at 16.51 195.58 0)
 			(effects
 				(font
@@
 		)
 		(property "Footprint" ""
-			(at 26.67 190.5 0)
+			(at 16.51 190.5 0)
 			(effects
 				(font
@@
 		)
 		(property "Datasheet" ""
-			(at 26.67 190.5 0)
+			(at 16.51 190.5 0)
 			(effects
 				(font
@@
 		)
 		(property "Description" "Power symbol creates a global label with name \"GND\" , ground"
-			(at 26.67 190.5 0)
+			(at 16.51 190.5 0)
 			(effects
 				(font
@@
 	(symbol
 		(lib_id "power:GND")
-		(at 34.29 190.5 0)
+		(at 24.13 190.5 0)
 		(unit 1)
 		(exclude_from_sim no)
@@
 		(fields_autoplaced yes)
 		(property "Reference" "#PWR03"
-			(at 34.29 196.85 0)
+			(at 24.13 196.85 0)
 			(effects
 				(font
@@
 		)
 		(property "Value" "GND"
-			(at 34.29 195.58 0)
+			(at 24.13 195.58 0)
 			(effects
 				(font
@@
 		)
 		(property "Footprint" ""
-			(at 34.29 190.5 0)
+			(at 24.13 190.5 0)
 			(effects
 				(font
@@
 		)
 		(property "Datasheet" ""
-			(at 34.29 190.5 0)
+			(at 24.13 190.5 0)
 			(effects
 				(font
@@
 		)
 		(property "Description" "Power symbol creates a global label with name \"GND\" , ground"
-			(at 34.29 190.5 0)
+			(at 24.13 190.5 0)
 			(effects
 				(font
@@
 	(symbol
 		(lib_id "Connector:USB_C_Receptacle_USB2.0_16P")
-		(at 34.29 167.64 0)
+		(at 24.13 167.64 0)
 		(unit 1)
 		(exclude_from_sim no)
@@
 		(on_board yes)
 		(dnp no)
-		(fields_autoplaced yes)
 		(property "Reference" "J7"
-			(at 34.29 144.78 0)
+			(at 24.13 144.78 0)
 			(effects
 				(font
@@
 		)
 		(property "Value" "USB_C_Receptacle_USB2.0_16P"
-			(at 34.29 147.32 0)
+			(at 28.194 147.066 0)
 			(effects
 				(font
@@
 		)
 		(property "Footprint" "Connector_USB:USB_C_Receptacle_GCT_USB4085"
-			(at 38.1 167.64 0)
+			(at 27.94 167.64 0)
 			(effects
 				(font
@@
 		)
 		(property "Datasheet" "https://www.usb.org/sites/default/files/documents/usb_type-c.zip"
-			(at 38.1 167.64 0)
+			(at 27.94 167.64 0)
 			(effects
 				(font
@@
 		)
 		(property "Description" "USB 2.0-only 16P Type-C Receptacle connector"
-			(at 34.29 167.64 0)
+			(at 24.13 167.64 0)
 			(effects
 				(font
@@
 		)
 		(property "LCSC" "C7095263"
-			(at 34.29 167.64 0)
+			(at 24.13 167.64 0)
 			(effects
 				(font
