File: sensor.kicad_sch (KiCad schematic)
At the start: 9 parts, among them J11 Register, J12 I2C_Source, J13 I2C_2, J14 I2C_3, J2 RegSense, J5 Conn_01x04_Pin, J6 I2C_1, U1 MH-Z19B

Commit message: fin
Parts:
- removed J11: Register, Connector_PinHeader_2.54mm:PinHeader_1x03_P2.54mm_Vertical, symbol Connector:Conn_01x03_Pin
- added J11: Reg2, Connector_PinSocket_2.54mm:PinSocket_1x02_P2.54mm_Vertical, symbol Connector:Conn_01x02_Pin
- added J17: Conn_01x04_Pin, Connector_PinHeader_2.54mm:PinHeader_1x04_P2.54mm_Vertical, symbol Connector:Conn_01x04_Pin
- added R2: 1k, Resistor_THT:R_Axial_DIN0207_L6.3mm_D2.5mm_P10.16mm_Horizontal, symbol Device:R
- J2: value RegSense -> Reg1
- R1: footprint Resistor_SMD:R_0603_1608Metric -> Resistor_THT:R_Axial_DIN0207_L6.3mm_D2.5mm_P10.16mm_Horizontal
Connections:
- net GND: now also J11.1 (Pin_1), J17.4 (Pin_4)
- net v3v: no longer R1.1
- net reg renamed adc1
- net adc1: now also J17.2 (Pin_2)
- new net adc2: J11.2 (Pin_2), J17.3 (Pin_3), R2.1
- new net adc_v3v: J17.1 (Pin_1), R1.1, R2.2
Other:
- moved on the sheet: J2

Commit message: update
Connections:
- net GND: now also J5.2 (Pin_2); no longer J5.4 (Pin_4)
- net UART(d2u) renamed TX(ESP_DOWN)
- net TX(ESP_DOWN): now also J5.3 (Pin_3); no longer J5.2 (Pin_2)
- net UART(u2d) renamed RX(ESP_UP)
- net RX(ESP_UP): now also J5.4 (Pin_4); no longer J5.3 (Pin_3)
Changed lines of the file:
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@@
+	(wire
+		(pts
+			(xy 52.07 64.77) (xy 52.07 72.39)
+		)
+		(stroke
+			(width 0)
+			(type default)
+		)
+	)
 	(wire
 		(pts
@@
 	(wire
 		(pts
-			(xy 45.72 67.31) (xy 54.61 67.31)
+			(xy 53.34 67.31) (xy 54.61 67.31)
 		)
 		(stroke
@@
 	(wire
 		(pts
-			(xy 43.18 74.93) (xy 33.02 74.93)
-		)
-		(stroke
-			(width 0)
-			(type default)
-		)
-	)
-	(wire
-		(pts
 			(xy 128.27 99.06) (xy 129.54 99.06)
 		)
@@
 	(wire
 		(pts
+			(xy 33.02 69.85) (xy 34.29 69.85)
+		)
+		(stroke
+			(width 0)
+			(type default)
+		)
+	)
+	(wire
+		(pts
 			(xy 113.03 86.36) (xy 134.62 86.36)
 		)
@@
 	(wire
 		(pts
+			(xy 34.29 69.85) (xy 34.29 78.74)
+		)
+		(stroke
+			(width 0)
+			(type default)
+		)
+	)
+	(wire
+		(pts
+			(xy 53.34 67.31) (xy 53.34 74.93)
+		)
+		(stroke
+			(width 0)
+			(type default)
+		)
+	)
+	(wire
+		(pts
 			(xy 86.36 115.57) (xy 97.79 115.57)
 		)
@@
 	(wire
 		(pts
-			(xy 45.72 72.39) (xy 45.72 67.31)
-		)
-		(stroke
-			(width 0)
-			(type default)
-		)
-	)
-	(wire
-		(pts
 			(xy 134.62 86.36) (xy 134.62 99.06)
 		)
@@
 	(wire
 		(pts
-			(xy 43.18 78.74) (xy 43.18 74.93)
-		)
-		(stroke
-			(width 0)
-			(type default)
-		)
-	)
-	(wire
-		(pts
-			(xy 41.91 64.77) (xy 54.61 64.77)
-		)
-		(stroke
-			(width 0)
-			(type default)
-		)
-	)
-	(wire
-		(pts
-			(xy 33.02 72.39) (xy 45.72 72.39)
+			(xy 33.02 74.93) (xy 53.34 74.93)
 		)
 		(stroke
@@
 	(wire
 		(pts
+			(xy 52.07 64.77) (xy 54.61 64.77)
+		)
+		(stroke
+			(width 0)
+			(type default)
+		)
+	)
+	(wire
+		(pts
 			(xy 134.62 86.36) (xy 152.4 86.36)
 		)
@@
 	(wire
 		(pts
+			(xy 33.02 72.39) (xy 52.07 72.39)
+		)
+		(stroke
+			(width 0)
+			(type default)
+		)
+	)
+	(wire
+		(pts
 			(xy 95.25 113.03) (xy 95.25 124.46)
 		)
@@
 	(wire
 		(pts
-			(xy 33.02 69.85) (xy 41.91 69.85)
-		)
-		(stroke
-			(width 0)
-			(type default)
-		)
-	)
-	(wire
-		(pts
 			(xy 33.02 67.31) (xy 36.83 67.31)
 		)
@@
 	(wire
 		(pts
-			(xy 43.18 78.74) (xy 64.77 78.74)
+			(xy 34.29 78.74) (xy 64.77 78.74)
 		)
 		(stroke
@@
 		(pts
 			(xy 137.16 99.06) (xy 137.16 78.74)
-		)
-		(stroke
-			(width 0)
-			(type default)
-		)
-	)
-	(wire
-		(pts
-			(xy 41.91 69.85) (xy 41.91 64.77)
 		)
 		(stroke
@@
 		)
 	)
-	(label "GND"
-		(at 40.64 74.93 0)
-		(fields_autoplaced yes)
-		(effects
-			(font
-				(size 1.27 1.27)
-			)
-			(justify left bottom)
-		)
-	)
-	(label "UART(d2u)"
-		(at 36.83 69.85 0)
-		(fields_autoplaced yes)
-		(effects
-			(font
-				(size 1.27 1.27)
-			)
-			(justify left bottom)
-		)
-	)
 	(label "adc2"
 		(at 114.3 83.82 0)
@@
 		)
 	)
+	(label "GND"
+		(at 52.07 78.74 0)
+		(fields_autoplaced yes)
+		(effects
+			(font
+				(size 1.27 1.27)
+			)
+			(justify left bottom)
+		)
+	)
 	(label "adc_v3v"
 		(at 118.11 78.74 180)
@@
 		)
 	)
+	(label "RX(ESP_UP)"
+		(at 38.1 74.93 0)
+		(fields_autoplaced yes)
+		(effects
+			(font
+				(size 1.27 1.27)
+			)
+			(justify left bottom)
+		)
+	)
+	(label "TX(ESP_DOWN)"
+		(at 36.83 72.39 0)
+		(fields_autoplaced yes)
+		(effects
+			(font
+				(size 1.27 1.27)
+			)
+			(justify left bottom)
+		)
+	)
 	(label "GND"
 		(at 114.3 86.36 0)
@@
 		(fields_autoplaced yes)
 		(effects
-			(font
-				(size 1.27 1.27)
-			)
-			(justify left bottom)
-		)
-	)
-	(label "UART(u2d)"
-		(at 35.56 72.39 0)
-		(fields_autoplaced yes)
-		(effects

Commit message: ok
Parts:
- renumbered J6 to J22
Changed lines of the file:
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@@
 		(dnp no)
 		(fields_autoplaced yes)
-		(property "Reference" "J6"
+		(property "Reference" "J22"
 			(at 73.66 132.08 90)
 			(effects
@@
 			(project "env_sensor"
 				(path "/f2c86898-5243-416b-bded-1093a29d5169/2c1791df-285c-4a68-8657-c16ce2e21da9"
-					(reference "J6")
+					(reference "J22")
 					(unit 1)
 				)

Commit message: update
Parts:
- removed J13: I2C_2, Connector_PinSocket_2.54mm:PinSocket_1x04_P2.54mm_Vertical, symbol Connector:Conn_01x04_Socket
- removed J14: I2C_3, Connector_PinSocket_2.54mm:PinSocket_1x04_P2.54mm_Vertical, symbol Connector:Conn_01x04_Socket
- removed J22: I2C_1, Connector_PinSocket_2.54mm:PinSocket_1x04_P2.54mm_Vertical, symbol Connector:Conn_01x04_Socket
- R1, R2: value 1k -> ~; now left out of the parts list

Commit message: update
Parts:
- removed J12: I2C_Source, Connector_PinHeader_2.54mm:PinHeader_1x04_P2.54mm_Vertical, symbol Connector:Conn_01x04_Pin
- added J8: Conn_01x08_Pin, Connector_PinHeader_2.54mm:PinHeader_2x04_P2.54mm_Vertical, symbol Connector:Conn_01x08_Pin
- U1: footprint mh-z19b:Winsen_MH-Z19B -> sensor_Carbon_dioxide:mh-z19b
Connections:
- net GND: now also J8.7 (Pin_7), J8.8 (Pin_8)
- net v3v: now also J8.1 (Pin_1)
- new net IO13: J8.3 (Pin_3)
- new net IO14: J8.4 (Pin_4)
- new net IO38: J8.2 (Pin_2)
- new net IO6: J8.5 (Pin_5)
- new net IO7: J8.6 (Pin_6)
Changed lines of the file:
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@@
+	(wire
+		(pts
+			(xy 43.18 115.57) (xy 55.88 115.57)
+		)
+		(stroke
+			(width 0)
+			(type default)
+		)
+	)
 	(wire
 		(pts
@@
 	(wire
 		(pts
+			(xy 43.18 118.11) (xy 55.88 118.11)
+		)
+		(stroke
+			(width 0)
+			(type default)
+		)
+	)
+	(wire
+		(pts
 			(xy 33.02 69.85) (xy 34.29 69.85)
 		)
@@
 	(wire
 		(pts
-			(xy 59.69 118.11) (xy 77.47 118.11)
-		)
-		(stroke
-			(width 0)
-			(type default)
-		)
-	)
-	(wire
-		(pts
 			(xy 129.54 81.28) (xy 129.54 99.06)
 		)
@@
 	(wire
 		(pts
+			(xy 43.18 113.03) (xy 55.88 113.03)
+		)
+		(stroke
+			(width 0)
+			(type default)
+		)
+	)
+	(wire
+		(pts
 			(xy 53.34 67.31) (xy 53.34 74.93)
 		)
@@
 	(wire
 		(pts
-			(xy 59.69 113.03) (xy 72.39 113.03)
+			(xy 43.18 123.19) (xy 55.88 123.19)
+		)
+		(stroke
+			(width 0)
+			(type default)
+		)
+	)
+	(wire
+		(pts
+			(xy 43.18 120.65) (xy 55.88 120.65)
 		)
 		(stroke
@@
 	(wire
 		(pts
-			(xy 59.69 115.57) (xy 74.93 115.57)
-		)
-		(stroke
-			(width 0)
-			(type default)
-		)
-	)
-	(wire
-		(pts
-			(xy 59.69 110.49) (xy 69.85 110.49)
+			(xy 43.18 128.27) (xy 55.88 128.27)
+		)
+		(stroke
+			(width 0)
+			(type default)
+		)
+	)
+	(wire
+		(pts
+			(xy 43.18 125.73) (xy 55.88 125.73)
 		)
 		(stroke
@@
 		(pts
 			(xy 52.07 64.77) (xy 54.61 64.77)
+		)
+		(stroke
+			(width 0)
+			(type default)
+		)
+	)
+	(wire
+		(pts
+			(xy 43.18 110.49) (xy 55.88 110.49)
 		)
 		(stroke
@@
 		)
 	)
-	(label "SDA"
-		(at 63.5 118.11 0)
+	(label "IO6"
+		(at 46.99 120.65 0)
+		(fields_autoplaced yes)
+		(effects
+			(font
+				(size 1.27 1.27)
+			)
+			(justify left bottom)
+		)
+	)
+	(label "v3v"
+		(at 46.99 110.49 0)
+		(fields_autoplaced yes)
+		(effects
+			(font
+				(size 1.27 1.27)
+			)
+			(justify left bottom)
+		)
+	)
+	(label "IO14"
+		(at 46.99 118.11 0)
+		(fields_autoplaced yes)
+		(effects
+			(font
+				(size 1.27 1.27)
+			)
+			(justify left bottom)
+		)
+	)
+	(label "IO13"
+		(at 46.99 115.57 0)
+		(fields_autoplaced yes)
+		(effects
+			(font
+				(size 1.27 1.27)
+			)
+			(justify left bottom)
+		)
+	)
+	(label "GND"
+		(at 46.99 128.27 0)
+		(fields_autoplaced yes)
+		(effects
+			(font
+				(size 1.27 1.27)
+			)
+			(justify left bottom)
+		)
+	)
+	(label "IO38"
+		(at 46.99 113.03 0)
 		(fields_autoplaced yes)
 		(effects
@@
 		)
 	)
+	(label "GND"
+		(at 46.99 125.73 0)
+		(fields_autoplaced yes)
+		(effects
+			(font
+				(size 1.27 1.27)
+			)
+			(justify left bottom)
+		)
+	)
 	(label "adc_v3v"
 		(at 118.11 78.74 180)
@@
 		)
 	)
-	(label "SCL"
-		(at 63.5 115.57 0)
-		(fields_autoplaced yes)
-		(effects
-			(font
-				(size 1.27 1.27)
-			)
-			(justify left bottom)
-		)
-	)
 	(label "RX(ESP_UP)"
 		(at 38.1 74.93 0)
@@
 		)
 	)
-	(label "v3v"
-		(at 63.5 110.49 0)
-		(fields_autoplaced yes)
-		(effects
-			(font
-				(size 1.27 1.27)
-			)
-			(justify left bottom)
-		)
-	)
 	(label "adc1"
 		(at 114.3 81.28 0)
@@
 		)
 	)
-	(label "GND"
-		(at 63.5 113.03 0)
+	(label "IO7"
+		(at 46.99 123.19 0)
 		(fields_autoplaced yes)
 		(effects
@@
 	)
 	(symbol
-		(lib_id "Connector:Conn_01x04_Pin")
-		(at 54.61 113.03 0)
-		(unit 1)
-		(exclude_from_sim no)
-		(in_bom no)
-		(on_board yes)
-		(dnp no)
-		(fields_autoplaced yes)
-		(property "Reference" "J12"
-			(at 55.245 105.41 0)
-			(effects
-				(font
-					(size 1.27 1.27)
-				)
-			)
-		)
-		(property "Value" "I2C_Source"
-			(at 55.245 107.95 0)
-			(effects
-				(font
-					(size 1.27 1.27)
-				)
-			)
-		)
-		(property "Footprint" "Connector_PinHeader_2.54mm:PinHeader_1x04_P2.54mm_Vertical"
-			(at 54.61 113.03 0)
-			(effects
-				(font
-					(size 1.27 1.27)
-				)
-				(hide yes)
-			)
-		)
-		(property "Datasheet" "~"
-			(at 54.61 113.03 0)
-			(effects
-				(font
-					(size 1.27 1.27)
-				)
-				(hide yes)
-			)
-		)
-		(property "Description" "Generic connector, single row, 01x04, script generated"
-			(at 54.61 113.03 0)
-			(effects
-				(font
-					(size 1.27 1.27)
-				)
-				(hide yes)
-			)
-		)
-		(pin "1"
-		)
-		(pin "4"
-		)
-		(pin "3"
-		)
-		(pin "2"
-		)
-		(instances
-			(project ""
-				(path "/f2c86898-5243-416b-bded-1093a29d5169/2c1791df-285c-4a68-8657-c16ce2e21da9"
-					(reference "J12")
-					(unit 1)
-				)
-			)
-		)
-	)
-	(symbol
 		(lib_id "Device:R")
 		(at 140.97 99.06 270)
@@
 	)
 	(symbol
+		(lib_id "Connector:Conn_01x08_Pin")
+		(at 38.1 118.11 0)
+		(unit 1)
+		(exclude_from_sim no)
+		(in_bom no)
+		(on_board yes)
+		(dnp no)
+		(property "Reference" "J8"
+			(at 38.735 105.41 0)
+			(effects
+				(font
+					(size 1.27 1.27)
+				)
+			)
+		)
+		(property "Value" "Conn_01x08_Pin"
+			(at 38.735 107.95 0)
+			(effects
+				(font
+					(size 1.27 1.27)
+				)
+			)
+		)
+		(property "Footprint" "Connector_PinHeader_2.54mm:PinHeader_2x04_P2.54mm_Vertical"
+			(at 45.466 133.096 0)
+			(effects
+				(font
+					(size 1.27 1.27)
+				)
+			)
+		)
+		(property "Datasheet" "~"
+			(at 38.1 118.11 0)
+			(effects
+				(font
+					(size 1.27 1.27)
+				)
+				(hide yes)
+			)
+		)
+		(property "Description" "Generic connector, single row, 01x08, script generated"
+			(at 38.1 118.11 0)
+			(effects
+				(font
+					(size 1.27 1.27)
+				)
+				(hide yes)
+			)
+		)
+		(pin "7"
+		)
+		(pin "6"
+		)
+		(pin "1"
+		)
+		(pin "2"
+		)
+		(pin "3"
+		)
+		(pin "4"
+		)
+		(pin "8"
+		)
+		(pin "5"
+		)
+		(instances
+			(project ""
+				(path "/f2c86898-5243-416b-bded-1093a29d5169/2c1791df-285c-4a68-8657-c16ce2e21da9"
+					(reference "J8")
+					(unit 1)
+				)
+			)
+		)
+	)
+	(symbol
 		(lib_id "mh_z19b:MH-Z19B")
 		(at 64.77 69.85 0)
@@
 			)
 		)
-		(property "Footprint" "mh-z19b:Winsen_MH-Z19B"
+		(property "Footprint" "sensor_Carbon_dioxide:mh-z19b"
 			(at 64.77 86.36 0)
 			(effects
